Commit message: joint1 working with MoveIt

File: catkin_ws/src/control/astra_description/urdf/astra.urdf.xacro (robot description, xacro)
@@ -209,5 +209,5 @@
 		<origin xyz="${base_link_attach_point}" />
 		<axis xyz="0 0 1"/>
-		<limit effort="1000" velocity="0.5" lower="${-(pi)}" upper="${pi}"/>
+		<limit effort="1000" velocity="2" lower="${-(pi)*2}" upper="${pi*2}"/>
 	</joint>
 	<!-- joint2 -->

Commit message: position control of motors now working with qc

File: catkin_ws/src/control/astra_description/urdf/astra.urdf.xacro (robot description, xacro)
@@ -209,5 +209,5 @@
 		<origin xyz="${base_link_attach_point}" />
 		<axis xyz="0 0 1"/>
-		<limit effort="1000" velocity="2" lower="${-(pi)*2}" upper="${pi*2}"/>
+		<limit effort="1000" velocity="0.5" lower="${-(pi)*2}" upper="${pi*2}"/>
 	</joint>
 	<!-- joint2 -->

Commit message: merge HD workspace on backup jetson

File: catkin_ws/src/control/astra_description/urdf/astra.urdf.xacro (robot description, xacro)
@@ -209,5 +209,5 @@
 		<origin xyz="${base_link_attach_point}" />
 		<axis xyz="0 0 1"/>
-		<limit effort="1000" velocity="0.5" lower="${-(pi)*2}" upper="${pi*2}"/>
+		<limit effort="1000" velocity="0.01" lower="${-(pi)*2}" upper="${pi*2}"/>
 	</joint>
 	<!-- joint2 -->

Commit message: robot config with the new urdf

File: catkin_ws/src/control/astra_description/urdf/astra.urdf.xacro (robot description, xacro)
@@ -3,61 +3,75 @@
 <!-- ======================================================================================================================== -->
 	<!-- ==========CONSANTS========== -->
+	<!-- base_link is rover -->
 	<!-- base_link constants -->
-	<xacro:property name="base_link_dim_x" value="0.3" />
-	<xacro:property name="base_link_dim_y" value="0.3" />
-	<xacro:property name="base_link_dim_z" value="0.1" />
-	<xacro:property name="base_link_dim" value="0.3 0.3 0.1" />
+	<xacro:property name="base_link_dim_x" value="0.6" />
+	<xacro:property name="base_link_dim_y" value="0.5" />
+	<xacro:property name="base_link_dim_z" value="0.16125" />
+	<xacro:property name="base_link_dim" value="0.6 0.5 0.16125" />
 	<xacro:property name="base_link_btm_shift_x" value="0" />
 	<xacro:property name="base_link_btm_shift_y" value="0" />
 	<xacro:property name="base_link_btm_shift_z" value="0" />
-	<xacro:property name="base_link_top_shift_x" value="0" />
+	<xacro:property name="base_link_top_shift_x" value="${(0.525-(base_link_dim_x/2))}" />
 	<xacro:property name="base_link_top_shift_y" value="0" />
 	<xacro:property name="base_link_top_shift_z" value="${(base_link_dim_z/2)}" />
 	<xacro:property name="base_link_origin" value="0 0 0" />
-	<xacro:property name="base_link_attach_point" value="0 0 ${((base_link_dim_z/2)+0)}" />
+	<xacro:property name="base_link_attach_point" value="${((0.525-(base_link_dim_x/2))+0)} 0 ${((base_link_dim_z/2)+0)}" />
 	<!-- link1 constants -->
-	<xacro:property name="link1_dim_x" value="0.083" />
-	<xacro:property name="link1_dim_y" value="0.156" />
-	<xacro:property name="link1_dim_z" value="0.14" />
-	<xacro:property name="link1_dim" value="0.083 0.156 0.14" />
+	<xacro:property name="link1_dim_x" value="0.08" />
+	<xacro:property name="link1_dim_y" value="0.1505" />
+	<xacro:property name="link1_dim_z" value="0.138" />
+	<xacro:property name="link1_dim" value="0.08 0.1505 0.138" />
 	<xacro:property name="link1_btm_shift_x" value="0" />
-	<xacro:property name="link1_btm_shift_y" value="0" />
+	<xacro:property name="link1_btm_shift_y" value="${-((0.094-(link1_dim_y/2)))}" />
 	<xacro:property name="link1_btm_shift_z" value="${(link1_dim_z/2)}" />
 	<xacro:property name="link1_top_shift_x" value="0" />
-	<xacro:property name="link1_top_shift_y" value="0" />
-	<xacro:property name="link1_top_shift_z" value="${((link1_dim_z/2)-0.05)}" />
-	<xacro:property name="link1_origin" value="0 0 ${(link1_dim_z/2)}" />
-	<xacro:property name="link1_attach_point" value="0 0 ${(((link1_dim_z/2)-0.05)+(link1_dim_z/2))}" />
+	<xacro:property name="link1_top_shift_y" value="${(link1_dim_x-0.0565)}" />
+	<xacro:property name="link1_top_shift_z" value="${(0.098-(link1_dim_z/2))}" />
+	<xacro:property name="link1_origin" value="0 ${-((0.094-(link1_dim_y/2)))} ${(link1_dim_z/2)}" />
+	<xacro:property name="link1_attach_point" value="0 ${((link1_dim_x-0.0565)+-((0.094-(link1_dim_y/2))))} ${((0.098-(link1_dim_z/2))+(link1_dim_z/2))}" />
 	<!-- link2 constants -->
 	<xacro:property name="link2_dim_x" value="0.096" />
-	<xacro:property name="link2_dim_y" value="0.062" />
-	<xacro:property name="link2_dim_z" value="0.425" />
-	<xacro:property name="link2_dim" value="0.096 0.062 0.425" />
+	<xacro:property name="link2_dim_y" value="0.07" />
+	<xacro:property name="link2_dim_z" value="0.487225" />
+	<xacro:property name="link2_dim" value="0.096 0.07 0.487225" />
 	<xacro:property name="link2_btm_shift_x" value="0" />
 	<xacro:property name="link2_btm_shift_y" value="0" />
 	<xacro:property name="link2_btm_shift_z" value="${-((0.048-(link2_dim_z/2)))}" />
-	<xacro:property name="link2_top_shift_x" value="${(0.03224-(link2_dim_x/2))}" />
+	<xacro:property name="link2_top_shift_x" value="${(0.039225-(link2_dim_x/2))}" />
 	<xacro:property name="link2_top_shift_y" value="0" />
-	<xacro:property name="link2_top_shift_z" value="${((link2_dim_z/2)-0.032224)}" />
+	<xacro:property name="link2_top_shift_z" value="${((link2_dim_z/2)-0.039225)}" />
 	<xacro:property name="link2_origin" value="0 0 ${-((0.048-(link2_dim_z/2)))}" />
-	<xacro:property name="link2_attach_point" value="${((0.03224-(link2_dim_x/2))+0)} 0 ${(((link2_dim_z/2)-0.032224)+-((0.048-(link2_dim_z/2))))}" />
+	<xacro:property name="link2_attach_point" value="${((0.039225-(link2_dim_x/2))+0)} 0 ${(((link2_dim_z/2)-0.039225)+-((0.048-(link2_dim_z/2))))}" />
+	<!-- motor_j3 constants -->
+	<xacro:property name="motor_j3_dim_x" value="0.09" />
+	<xacro:property name="motor_j3_dim_y" value="0.07" />
+	<xacro:property name="motor_j3_dim_z" value="0.3" />
+	<xacro:property name="motor_j3_dim" value="0.09 0.07 0.3" />
+	<xacro:property name="motor_j3_btm_shift_x" value="-0.084225" />
+	<xacro:property name="motor_j3_btm_shift_y" value="0" />
+	<xacro:property name="motor_j3_btm_shift_z" value="0.004388" />
+	<xacro:property name="motor_j3_top_shift_x" value="0" />
+	<xacro:property name="motor_j3_top_shift_y" value="0" />
+	<xacro:property name="motor_j3_top_shift_z" value="0" />
+	<xacro:property name="motor_j3_origin" value="-0.084225 0 0.004388" />
+	<xacro:property name="motor_j3_attach_point" value="-0.084225 0 0.004388" />
 	<!-- link3 constants -->
-	<xacro:property name="link3_dim_x" value="0.092" />
+	<xacro:property name="link3_dim_x" value="0.115" />
 	<xacro:property name="link3_dim_y" value="0.112" />
-	<xacro:property name="link3_dim_z" value="0.334" />
-	<xacro:property name="link3_dim" value="0.092 0.112 0.334" />
-	<xacro:property name="link3_btm_shift_x" value="${(0.01615-(link3_dim_x/2))}" />
+	<xacro:property name="link3_dim_z" value="0.387" />
+	<xacro:property name="link3_dim" value="0.115 0.112 0.387" />
+	<xacro:property name="link3_btm_shift_x" value="${(0.02-(link3_dim_x/2))}" />
 	<xacro:property name="link3_btm_shift_y" value="0" />
-	<xacro:property name="link3_btm_shift_z" value="${-((0.096328-(link3_dim_z/2)))}" />
-	<xacro:property name="link3_top_shift_x" value="${-((0.0415-(link3_dim_x/2)))}" />
+	<xacro:property name="link3_btm_shift_z" value="${-((0.087-(link3_dim_z/2)))}" />
+	<xacro:property name="link3_top_shift_x" value="${(0.0415-(link3_dim_x/2))}" />
 	<xacro:property name="link3_top_shift_y" value="0" />
 	<xacro:property name="link3_top_shift_z" value="${(link3_dim_z/2)}" />
-	<xacro:property name="link3_origin" value="${(0.01615-(link3_dim_x/2))} 0 ${-((0.096328-(link3_dim_z/2)))}" />
-	<xacro:property name="link3_attach_point" value="${(-((0.0415-(link3_dim_x/2)))+(0.01615-(link3_dim_x/2)))} 0 ${((link3_dim_z/2)+-((0.096328-(link3_dim_z/2))))}" />
+	<xacro:property name="link3_origin" value="${(0.02-(link3_dim_x/2))} 0 ${-((0.087-(link3_dim_z/2)))}" />
+	<xacro:property name="link3_attach_point" value="${((0.0415-(link3_dim_x/2))+(0.02-(link3_dim_x/2)))} 0 ${((link3_dim_z/2)+-((0.087-(link3_dim_z/2))))}" />
 	<!-- link4 constants -->
 	<xacro:property name="link4_dim_x" value="0.08" />
-	<xacro:property name="link4_dim_y" value="0.173" />
-	<xacro:property name="link4_dim_z" value="0.12" />
-	<xacro:property name="link4_dim" value="0.08 0.173 0.12" />
+	<xacro:property name="link4_dim_y" value="0.175" />
+	<xacro:property name="link4_dim_z" value="0.1208" />
+	<xacro:property name="link4_dim" value="0.08 0.175 0.1208" />
 	<xacro:property name="link4_btm_shift_x" value="0" />
 	<xacro:property name="link4_btm_shift_y" value="0" />
@@ -65,33 +79,59 @@
 	<xacro:property name="link4_top_shift_x" value="0" />
 	<xacro:property name="link4_top_shift_y" value="0" />
-	<xacro:property name="link4_top_shift_z" value="${((link4_dim_z/2)-0.029)}" />
+	<xacro:property name="link4_top_shift_z" value="${((link4_dim_z/2)-0.031)}" />
 	<xacro:property name="link4_origin" value="0 0 ${(link4_dim_z/2)}" />
-	<xacro:property name="link4_attach_point" value="0 0 ${(((link4_dim_z/2)-0.029)+(link4_dim_z/2))}" />
+	<xacro:property name="link4_attach_point" value="0 0 ${(((link4_dim_z/2)-0.031)+(link4_dim_z/2))}" />
 	<!-- link5 constants -->
-	<xacro:property name="link5_dim_x" value="0.047" />
-	<xacro:property name="link5_dim_y" value="0.056" />
-	<xacro:property name="link5_dim_z" value="0.08625" />
-	<xacro:property name="link5_dim" value="0.047 0.056 0.08625" />
+	<xacro:property name="link5_dim_x" value="0.045" />
+	<xacro:property name="link5_dim_y" value="0.045" />
+	<xacro:property name="link5_dim_z" value="0.09455" />
+	<xacro:property name="link5_dim" value="0.045 0.045 0.09455" />
 	<xacro:property name="link5_btm_shift_x" value="0" />
 	<xacro:property name="link5_btm_shift_y" value="0" />
-	<xacro:property name="link5_btm_shift_z" value="${((link5_dim_z/2)-0.0235)}" />
+	<xacro:property name="link5_btm_shift_z" value="${((link5_dim_z/2)-0.0318)}" />
 	<xacro:property name="link5_top_shift_x" value="0" />
 	<xacro:property name="link5_top_shift_y" value="0" />
 	<xacro:property name="link5_top_shift_z" value="${(link5_dim_z/2)}" />
-	<xacro:property name="link5_origin" value="0 0 ${((link5_dim_z/2)-0.0235)}" />
-	<xacro:property name="link5_attach_point" value="0 0 ${((link5_dim_z/2)+((link5_dim_z/2)-0.0235))}" />
+	<xacro:property name="link5_origin" value="0 0 ${((link5_dim_z/2)-0.0318)}" />
+	<xacro:property name="link5_attach_point" value="0 0 ${((link5_dim_z/2)+((link5_dim_z/2)-0.0318))}" />
 	<!-- gripper_base constants -->
-	<xacro:property name="gripper_base_dim_x" value="0.1196" />
-	<xacro:property name="gripper_base_dim_y" value="0.1105" />
-	<xacro:property name="gripper_base_dim_z" value="0.062" />
-	<xacro:property name="gripper_base_dim" value="0.1196 0.1105 0.062" />
-	<xacro:property name="gripper_base_btm_shift_x" value="${((gripper_base_dim_x/2)-0.03)}" />
-	<xacro:property name="gripper_base_btm_shift_y" value="0" />
+	<xacro:property name="gripper_base_dim_x" value="0.1565" />
+	<xacro:property name="gripper_base_dim_y" value="0.125" />
+	<xacro:property name="gripper_base_dim_z" value="0.103" />
+	<xacro:property name="gripper_base_dim" value="0.1565 0.125 0.103" />
+	<xacro:property name="gripper_base_btm_shift_x" value="${((gripper_base_dim_x/2)-0.076)}" />
+	<xacro:property name="gripper_base_btm_shift_y" value="${-((0.0671-(gripper_base_dim_y/2)))}" />
 	<xacro:property name="gripper_base_btm_shift_z" value="${(gripper_base_dim_z/2)}" />
-	<xacro:property name="gripper_base_top_shift_x" value="0" />
-	<xacro:property name="gripper_base_top_shift_y" value="0" />
-	<xacro:property name="gripper_base_top_shift_z" value="0" />
-	<xacro:property name="gripper_base_origin" value="${((gripper_base_dim_x/2)-0.03)} 0 ${(gripper_base_dim_z/2)}" />
-	<xacro:property name="gripper_base_attach_point" value="${(((gripper_base_dim_x/2)-0.03)+0)} 0 ${((gripper_base_dim_z/2)+0)}" />
+	<xacro:property name="gripper_base_top_shift_x" value="${-(((gripper_base_dim_x/2)-0.076))}" />
+	<xacro:property name="gripper_base_top_shift_y" value="${(0.0671-(gripper_base_dim_y/2))}" />
+	<xacro:property name="gripper_base_top_shift_z" value="${(gripper_base_dim_z/2)}" />
+	<xacro:property name="gripper_base_origin" value="${((gripper_base_dim_x/2)-0.076)} ${-((0.0671-(gripper_base_dim_y/2)))} ${(gripper_base_dim_z/2)}" />
+	<xacro:property name="gripper_base_attach_point" value="${(-(((gripper_base_dim_x/2)-0.076))+((gripper_base_dim_x/2)-0.076))} ${((0.0671-(gripper_base_dim_y/2))+-((0.0671-(gripper_base_dim_y/2))))} ${((gripper_base_dim_z/2)+(gripper_base_dim_z/2))}" />
+	<!-- gripper_left_finger constants -->
+	<xacro:property name="gripper_left_finger_dim_x" value="0.0215" />
+	<xacro:property name="gripper_left_finger_dim_y" value="0.016" />
+	<xacro:property name="gripper_left_finger_dim_z" value="0.045" />
+	<xacro:property name="gripper_left_finger_dim" value="0.0215 0.016 0.045" />
+	<xacro:property name="gripper_left_finger_btm_shift_x" value="0" />
+	<xacro:property name="gripper_left_finger_btm_shift_y" value="${(gripper_left_finger_dim_y/2)}" />
+	<xacro:property name="gripper_left_finger_btm_shift_z" value="${(gripper_left_finger_dim_z/2)}" />
+	<xacro:property name="gripper_left_finger_top_shift_x" value="0" />
+	<xacro:property name="gripper_left_finger_top_shift_y" value="0" />
+	<xacro:property name="gripper_left_finger_top_shift_z" value="0" />
+	<xacro:property name="gripper_left_finger_origin" value="0 ${(gripper_left_finger_dim_y/2)} ${(gripper_left_finger_dim_z/2)}" />
+	<xacro:property name="gripper_left_finger_attach_point" value="0 ${((gripper_left_finger_dim_y/2)+0)} ${((gripper_left_finger_dim_z/2)+0)}" />
+	<!-- gripper_right_finger constants -->
+	<xacro:property name="gripper_right_finger_dim_x" value="0.0215" />
+	<xacro:property name="gripper_right_finger_dim_y" value="0.016" />
+	<xacro:property name="gripper_right_finger_dim_z" value="0.045" />
+	<xacro:property name="gripper_right_finger_dim" value="0.0215 0.016 0.045" />
+	<xacro:property name="gripper_right_finger_btm_shift_x" value="0" />
+	<xacro:property name="gripper_right_finger_btm_shift_y" value="${(-(gripper_right_finger_dim_y)/2)}" />
+	<xacro:property name="gripper_right_finger_btm_shift_z" value="${(gripper_right_finger_dim_z/2)}" />
+	<xacro:property name="gripper_right_finger_top_shift_x" value="0" />
+	<xacro:property name="gripper_right_finger_top_shift_y" value="0" />
+	<xacro:property name="gripper_right_finger_top_shift_z" value="0" />
+	<xacro:property name="gripper_right_finger_origin" value="0 ${(-(gripper_right_finger_dim_y)/2)} ${(gripper_right_finger_dim_z/2)}" />
+	<xacro:property name="gripper_right_finger_attach_point" value="0 ${((-(gripper_right_finger_dim_y)/2)+0)} ${((gripper_right_finger_dim_z/2)+0)}" />
 	<!-- ======================================================================================================================== -->
 	<!-- ==========LINKS========== -->
@@ -141,4 +181,19 @@
 		</collision>
 	</link>
+	<!-- motor_j3 -->
+	<link name="motor_j3">
+		<visual>
+			<geometry>
+				<box size="${motor_j3_dim}"/>
+			</geometry>
+			<origin xyz="${motor_j3_origin}" />
+		</visual>
+		<collision>
+			<geometry>
+				<box size="${motor_j3_dim}"/>
+			</geometry>
+			<origin xyz="${motor_j3_origin}" />
+		</collision>
+	</link>
 	<!-- link3 -->
 	<link name="link3">
@@ -199,4 +254,34 @@
 			</geometry>
 			<origin xyz="${gripper_base_origin}" />
+		</collision>
+	</link>
+	<!-- gripper_left_finger -->
+	<link name="gripper_left_finger">
+		<visual>
+			<geometry>
+				<box size="${gripper_left_finger_dim}"/>
+			</geometry>
+			<origin xyz="${gripper_left_finger_origin}" />
+		</visual>
+		<collision>
+			<geometry>
+				<box size="${gripper_left_finger_dim}"/>
+			</geometry>
+			<origin xyz="${gripper_left_finger_origin}" />
+		</collision>
+	</link>
+	<!-- gripper_right_finger -->
+	<link name="gripper_right_finger">
+		<visual>
+			<geometry>
+				<box size="${gripper_right_finger_dim}"/>
+			</geometry>
+			<origin xyz="${gripper_right_finger_origin}" />
+		</visual>
+		<collision>
+			<geometry>
+				<box size="${gripper_right_finger_dim}"/>
+			</geometry>
+			<origin xyz="${gripper_right_finger_origin}" />
 		</collision>
 	</link>
@@ -209,5 +294,5 @@
 		<origin xyz="${base_link_attach_point}" />
 		<axis xyz="0 0 1"/>
-		<limit effort="1000" velocity="0.01" lower="${-(pi)*2}" upper="${pi*2}"/>
+		<limit effort="1" velocity="0.5" lower="${(pi*-2)}" upper="${(pi*2)}"/>
 	</joint>
 	<!-- joint2 -->
@@ -217,5 +302,13 @@
 		<origin xyz="${link1_attach_point}" />
 		<axis xyz="0 1 0"/>
-		<limit effort="1000" velocity="0.5" lower="${-(pi)}" upper="${pi}"/>
+		<limit effort="1" velocity="0.5" lower="-1.34" upper="2.07"/>
+	</joint>
+	<!-- motor_j3_joint -->
+	<joint name="motor_j3_joint" type="fixed">
+		<parent link="link2"/>
+		<child link="motor_j3"/>
+		<origin xyz="${link2_attach_point}" />
+		<axis xyz="1 0 0"/>
+		<limit effort="1" velocity="0.5" lower="${-(pi)}" upper="${pi}"/>
 	</joint>
 	<!-- joint3 -->
@@ -223,7 +316,7 @@
 		<parent link="link2"/>
 		<child link="link3"/>
-		<origin xyz="${link2_attach_point}" />
-		<axis xyz="0 1 0"/>
-		<limit effort="1000" velocity="0.5" lower="${-(pi)}" upper="${pi}"/>
+		<origin xyz="${link2_attach_point}" rpy="0 ${pi/2} 0" />
+		<axis xyz="0 1 0"/>
+		<limit effort="1" velocity="0.5" lower="-1.1" upper="1"/>
 	</joint>
 	<!-- joint4 -->
@@ -233,5 +326,5 @@
 		<origin xyz="${link3_attach_point}" />
 		<axis xyz="0 0 1"/>
-		<limit effort="1000" velocity="0.5" lower="${-(pi)}" upper="${pi}"/>
+		<limit effort="1" velocity="0.5" lower="${(pi*-2)}" upper="${(pi*2)}"/>
 	</joint>
 	<!-- joint5 -->
@@ -241,5 +334,5 @@
 		<origin xyz="${link4_attach_point}" />
 		<axis xyz="0 1 0"/>
-		<limit effort="1000" velocity="0.5" lower="${-(pi)}" upper="${pi}"/>
+		<limit effort="1" velocity="0.5" lower="-1.9" upper="1.9"/>
 	</joint>
 	<!-- joint6 -->
@@ -249,5 +342,22 @@
 		<origin xyz="${link5_attach_point}" />
 		<axis xyz="0 0 1"/>
-		<limit effort="1000" velocity="0.5" lower="${-(pi)}" upper="${pi}"/>
+		<limit effort="1" velocity="0.5" lower="${-(pi)}" upper="${pi}"/>
+	</joint>
+	<!-- gripper_left_finger_joint -->
+	<joint name="gripper_left_finger_joint" type="prismatic">
+		<parent link="gripper_base"/>
+		<child link="gripper_left_finger"/>
+		<origin xyz="${gripper_base_attach_point}" />
+		<axis xyz="0 1 0"/>
+		<limit effort="1" velocity="0.5" lower="0" upper="0.04"/>
+	</joint>
+	<!-- gripper_right_finger_joint -->
+	<joint name="gripper_right_finger_joint" type="prismatic">
+		<parent link="gripper_base"/>
+		<child link="gripper_right_finger"/>
+		<origin xyz="${gripper_base_attach_point}" />
+		<axis xyz="0 1 0"/>
+		<limit effort="1" velocity="0.5" lower="0" upper="0.1"/>
+		<mimic joint="gripper_left_finger_joint" multiplier="-1" offset="0"/>
 	</joint>
 </robot>
