Commit message: ready to test ik

File: catkin_ws/src/control/urdf_creator/astra.urdf.xacro (robot description, xacro)
@@ -294,5 +294,5 @@
 		<origin xyz="${base_link_attach_point}" />
 		<axis xyz="0 0 1"/>
-		<limit effort="10" velocity="0.2" lower="${(pi*-2)}" upper="${(pi*2)}"/>
+		<limit effort="1" velocity="0.5" lower="${(pi*-2)}" upper="${(pi*2)}"/>
 	</joint>
 	<!-- joint2 -->
@@ -302,5 +302,5 @@
 		<origin xyz="${link1_attach_point}" />
 		<axis xyz="0 1 0"/>
-		<limit effort="10" velocity="0.2" lower="-1.34" upper="2.07"/>
+		<limit effort="1" velocity="0.5" lower="-1.34" upper="2.07"/>
 	</joint>
 	<!-- motor_j3_joint -->
@@ -310,5 +310,5 @@
 		<origin xyz="${link2_attach_point}" />
 		<axis xyz="1 0 0"/>
-		<limit effort="1" velocity="0.2" lower="${-(pi)}" upper="${pi}"/>
+		<limit effort="1" velocity="0.5" lower="${-(pi)}" upper="${pi}"/>
 	</joint>
 	<!-- joint3 -->
@@ -318,5 +318,5 @@
 		<origin xyz="${link2_attach_point}" rpy="0 ${pi/2} 0" />
 		<axis xyz="0 1 0"/>
-		<limit effort="10" velocity="0.2" lower="-1.1" upper="1"/>
+		<limit effort="1" velocity="0.5" lower="-1.1" upper="1"/>
 	</joint>
 	<!-- joint4 -->
@@ -326,5 +326,5 @@
 		<origin xyz="${link3_attach_point}" />
 		<axis xyz="0 0 1"/>
-		<limit effort="10" velocity="0.2" lower="${(pi*-2)}" upper="${(pi*2)}"/>
+		<limit effort="1" velocity="0.5" lower="${(pi*-2)}" upper="${(pi*2)}"/>
 	</joint>
 	<!-- joint5 -->
@@ -334,5 +334,5 @@
 		<origin xyz="${link4_attach_point}" />
 		<axis xyz="0 1 0"/>
-		<limit effort="10" velocity="0.2" lower="-1.9" upper="1.9"/>
+		<limit effort="1" velocity="0.5" lower="-1.9" upper="1.9"/>
 	</joint>
 	<!-- joint6 -->
@@ -342,5 +342,5 @@
 		<origin xyz="${link5_attach_point}" />
 		<axis xyz="0 0 1"/>
-		<limit effort="10" velocity="0.2" lower="${-(pi)}" upper="${pi}"/>
+		<limit effort="1" velocity="0.5" lower="${-(pi)}" upper="${pi}"/>
 	</joint>
 	<!-- gripper_left_finger_joint -->
